File: Schematics/LineaMeta/LineaMeta.kicad_sch (KiCad schematic)
At the start: 7 parts, among them J1 Conn_02x08_Top_Bottom, Q1 BPW40

Commit message: Working basic version
Parts:
- removed R3, R4: R, symbol Device:R
- added J2: Pantalla, symbol Connector_Generic:Conn_01x04
Connections:
- net +3V3: now also J2.2 (Pin_2)
- net GND: now also J2.1 (Pin_1)
- net SCL: now also J2.3 (Pin_3)
- net SDA: now also J2.4 (Pin_4)
- net IR_INPUT: now reaches Q1.1 (C), R2.2
